Commit message: feat: Camera added to robot_description

File: urdf/panda_arm.urdf.xacro (robot description, xacro)
@@ -14,4 +14,67 @@
     <xacro:include filename="$(find aescape_panda_simulator)/urdf/panda.transmission.xacro"/>
     <xacro:panda_transmission robot_name="$(arg robot_name)"/>
+    <link name="$(arg robot_name)_camera">
+      <visual>
+        <geometry>
+          <box size="0.04 0.18 0.047"/>
+        </geometry>
+      </visual>
+      <collision>
+        <geometry>
+          <box size="0.04 0.18 0.047"/>
+        </geometry>
+      </collision>
+      <inertial>
+        <mass value="0.2"/>
+        <inertia ixx="1.0" ixy="0.0" ixz="0.0" iyy="1.0" iyz="0.0" izz="1.0"/>
+      </inertial>
+    </link>
+    <joint name="camera_to_world" type="fixed">
+      <parent link="world" />
+      <child link="$(arg robot_name)_camera" />
+      <origin xyz="1.0 $(arg origin_y) 1.0" rpy="0.0 0.7854 3.1416" />
+      <dynamics damping="1.0"/>
+    </joint>
+    <gazebo reference="$(arg robot_name)_camera">
+      <sensor name="$camera" type="depth">
+        <update_rate>20</update_rate>
+        <camera>
+          <horizontal_fov>1.047198</horizontal_fov>
+          <image>
+            <width>640</width>
+            <height>480</height>
+            <format>R8G8B8</format>
+          </image>
+          <clip>
+            <near>0.05</near>
+            <far>3</far>
+          </clip>
+        </camera>
+        <plugin name="camera_controller" filename="libgazebo_ros_openni_kinect.so">
+          <baseline>0.2</baseline>
+          <alwaysOn>true</alwaysOn>
+          <updateRate>1.0</updateRate>
+          <cameraName>$(arg robot_name)_camera_ir</cameraName>
+          <imageTopicName>/$(arg robot_name)/camera/color/image_raw</imageTopicName>
+          <cameraInfoTopicName>/$(arg robot_name)/camera/color/camera_info</cameraInfoTopicName>
+          <depthImageTopicName>/$(arg robot_name)/camera/depth/image_raw</depthImageTopicName>
+          <depthImageInfoTopicName>/$(arg robot_name)/camera/depth/camera_info</depthImageInfoTopicName>
+          <pointCloudTopicName>/$(arg robot_name)/camera/depth/points</pointCloudTopicName>
+          <frameName>$(arg robot_name)_camera</frameName>
+          <pointCloudCutoff>0.5</pointCloudCutoff>
+          <pointCloudCutoffMax>3.0</pointCloudCutoffMax>
+          <distortionK1>0.00000001</distortionK1>
+          <distortionK2>0.00000001</distortionK2>
+          <distortionK3>0.00000001</distortionK3>
+          <distortionT1>0.00000001</distortionT1>
+          <distortionT2>0.00000001</distortionT2>
+          <CxPrime>0</CxPrime>
+          <Cx>0</Cx>
+          <Cy>0</Cy>
+          <focalLength>0</focalLength>
+          <hackBaseline>0</hackBaseline>
+        </plugin>
+      </sensor>
+    </gazebo>
   </xacro:if>
 </robot>

Commit message: feat: Kinect visual added and rviz camera setup

File: urdf/panda_arm.urdf.xacro (robot description, xacro)
@@ -16,6 +16,9 @@
     <link name="$(arg robot_name)_camera">
       <visual>
+        <!--geometry>
+          <box size="0.04 0.18 0.047"/>
+        </geometry-->
         <geometry>
-          <box size="0.04 0.18 0.047"/>
+          <mesh filename="package://aescape_panda_simulator/meshes/visual/kinect.dae"/>
         </geometry>
       </visual>
@@ -38,5 +41,5 @@
     <gazebo reference="$(arg robot_name)_camera">
       <sensor name="$camera" type="depth">
-        <update_rate>20</update_rate>
+        <update_rate>10</update_rate>
         <camera>
           <horizontal_fov>1.047198</horizontal_fov>

Commit message: feat: depth_camera urdf and xacro done

File: urdf/panda_arm.urdf.xacro (robot description, xacro)
@@ -14,70 +14,6 @@
     <xacro:include filename="$(find aescape_panda_simulator)/urdf/panda.transmission.xacro"/>
     <xacro:panda_transmission robot_name="$(arg robot_name)"/>
-    <link name="$(arg robot_name)_camera">
-      <visual>
-        <!--geometry>
-          <box size="0.04 0.18 0.047"/>
-        </geometry-->
-        <geometry>
-          <mesh filename="package://aescape_panda_simulator/meshes/visual/kinect.dae"/>
-        </geometry>
-      </visual>
-      <collision>
-        <geometry>
-          <box size="0.04 0.18 0.047"/>
-        </geometry>
-      </collision>
-      <inertial>
-        <mass value="0.2"/>
-        <inertia ixx="1.0" ixy="0.0" ixz="0.0" iyy="1.0" iyz="0.0" izz="1.0"/>
-      </inertial>
-    </link>
-    <joint name="camera_to_world" type="fixed">
-      <parent link="world" />
-      <child link="$(arg robot_name)_camera" />
-      <origin xyz="1.0 $(arg origin_y) 1.0" rpy="0.0 0.7854 3.1416" />
-      <dynamics damping="1.0"/>
-    </joint>
-    <gazebo reference="$(arg robot_name)_camera">
-      <sensor name="$camera" type="depth">
-        <update_rate>10</update_rate>
-        <camera>
-          <horizontal_fov>1.047198</horizontal_fov>
-          <image>
-            <width>640</width>
-            <height>480</height>
-            <format>R8G8B8</format>
-          </image>
-          <clip>
-            <near>0.05</near>
-            <far>3</far>
-          </clip>
-        </camera>
-        <plugin name="camera_controller" filename="libgazebo_ros_openni_kinect.so">
-          <baseline>0.2</baseline>
-          <alwaysOn>true</alwaysOn>
-          <updateRate>1.0</updateRate>
-          <cameraName>$(arg robot_name)_camera_ir</cameraName>
-          <imageTopicName>/$(arg robot_name)/camera/color/image_raw</imageTopicName>
-          <cameraInfoTopicName>/$(arg robot_name)/camera/color/camera_info</cameraInfoTopicName>
-          <depthImageTopicName>/$(arg robot_name)/camera/depth/image_raw</depthImageTopicName>
-          <depthImageInfoTopicName>/$(arg robot_name)/camera/depth/camera_info</depthImageInfoTopicName>
-          <pointCloudTopicName>/$(arg robot_name)/camera/depth/points</pointCloudTopicName>
-          <frameName>$(arg robot_name)_camera</frameName>
-          <pointCloudCutoff>0.5</pointCloudCutoff>
-          <pointCloudCutoffMax>3.0</pointCloudCutoffMax>
-          <distortionK1>0.00000001</distortionK1>
-          <distortionK2>0.00000001</distortionK2>
-          <distortionK3>0.00000001</distortionK3>
-          <distortionT1>0.00000001</distortionT1>
-          <distortionT2>0.00000001</distortionT2>
-          <CxPrime>0</CxPrime>
-          <Cx>0</Cx>
-          <Cy>0</Cy>
-          <focalLength>0</focalLength>
-          <hackBaseline>0</hackBaseline>
-        </plugin>
-      </sensor>
-    </gazebo>
+    <xacro:include filename="$(find aescape_panda_simulator)/urdf/depth_camera.xacro"/>
+    <xacro:depth_camera camera_name="$(arg robot_name)" connected_to="world" xyz="1.0 $(arg origin_y) 1.0" rpy="0.0 0.7854 3.1416"/>
   </xacro:if>
 </robot>

Commit message: feat: using single robot_description to rviz and namespace/robot_description for controllers

File: urdf/panda_arm.urdf.xacro (robot description, xacro)
@@ -4,10 +4,11 @@
   <xacro:arg name="load_gazebo" default="false"/>
   <xacro:arg name="origin_y" default="0.0"/>
+  <link name="world"/>
   <xacro:include filename="$(find aescape_panda_simulator)/urdf/panda_arm.xacro"/>
   <xacro:unless value="$(arg load_gazebo)">
-    <xacro:panda_arm arm_id="$(arg robot_name)" xyz="0.0 $(arg origin_y) 0.0"/>
+    <xacro:panda_arm arm_id="$(arg robot_name)" connected_to="world" xyz="0.0 $(arg origin_y) 0.0"/>
   </xacro:unless>
   <xacro:if value="$(arg load_gazebo)">
-    <xacro:panda_arm in_gazebo="true" arm_id="$(arg robot_name)" xyz="0.0 $(arg origin_y) 0.0"/>
+    <xacro:panda_arm in_gazebo="true" connected_to="world" arm_id="$(arg robot_name)" xyz="0.0 $(arg origin_y) 0.0"/>
     <xacro:include filename="$(find aescape_panda_simulator)/urdf/panda.gazebo.xacro"/>
     <xacro:panda_gazebo robot_name="$(arg robot_name)"/>

File: urdf/panda_arm.xacro (robot description, xacro)
@@ -9,5 +9,5 @@
       </joint>
     </xacro:unless>
-    <xacro:property name="joint_damping" value="1.0"/>
+    <!--xacro:property name="joint_damping" value="1.0"/>
     <xacro:unless value="${in_gazebo == 'false'}">
       <link name="world" />
@@ -18,5 +18,5 @@
         <dynamics damping="${joint_damping}"/>
       </joint>
-    </xacro:unless>
+    </xacro:unless-->
     <link name="${arm_id}_link0">
       <visual>
