Commit message: feat: project name changed to aescape_gazebo

File: urdf/depth_camera.urdf.xacro (robot description, xacro)
@@ -1,5 +1,5 @@
 <?xml version="1.0"?>
 <robot xmlns:xacro="http://www.ros.org/wiki/xacro" name="panda">
-  <xacro:include filename="$(find aescape_panda_simulator)/urdf/depth_camera.xacro"/>
+  <xacro:include filename="$(find aescape_gazebo)/urdf/depth_camera.xacro"/>
   <xacro:depth_camera camera_name="camera" xyz="0 0 0.1" rpy="0.0 0.0 0.0"/>
 </robot>

File: urdf/depth_camera.xacro (robot description, xacro)
@@ -8,5 +8,5 @@
         </geometry>
         <!--geometry>
-          <mesh filename="package://aescape_panda_simulator/meshes/visual/kinect.dae"/>
+          <mesh filename="package://aescape_gazebo/meshes/visual/kinect.dae"/>
         </geometry-->
       </visual>

File: urdf/panda_arm.urdf.xacro (robot description, xacro)
@@ -5,5 +5,5 @@
   <xacro:arg name="origin_y" default="0.0"/>
   <link name="world"/>
-  <xacro:include filename="$(find aescape_panda_simulator)/urdf/panda_arm.xacro"/>
+  <xacro:include filename="$(find aescape_gazebo)/urdf/panda_arm.xacro"/>
   <xacro:unless value="$(arg load_gazebo)">
     <xacro:panda_arm arm_id="$(arg robot_name)" connected_to="world" xyz="0.0 $(arg origin_y) 0.0"/>
@@ -11,9 +11,9 @@
   <xacro:if value="$(arg load_gazebo)">
     <xacro:panda_arm in_gazebo="true" connected_to="world" arm_id="$(arg robot_name)" xyz="0.0 $(arg origin_y) 0.0"/>
-    <xacro:include filename="$(find aescape_panda_simulator)/urdf/panda.gazebo.xacro"/>
+    <xacro:include filename="$(find aescape_gazebo)/urdf/panda.gazebo.xacro"/>
     <xacro:panda_gazebo robot_name="$(arg robot_name)"/>
-    <xacro:include filename="$(find aescape_panda_simulator)/urdf/panda.transmission.xacro"/>
+    <xacro:include filename="$(find aescape_gazebo)/urdf/panda.transmission.xacro"/>
     <xacro:panda_transmission robot_name="$(arg robot_name)"/>
-    <xacro:include filename="$(find aescape_panda_simulator)/urdf/depth_camera.xacro"/>
+    <xacro:include filename="$(find aescape_gazebo)/urdf/depth_camera.xacro"/>
     <xacro:depth_camera camera_name="$(arg robot_name)" connected_to="world" xyz="1.0 $(arg origin_y) 1.0" rpy="0.0 0.7854 3.1416"/>
   </xacro:if>

File: urdf/panda_arm.xacro (robot description, xacro)
@@ -1,5 +1,5 @@
 <?xml version='1.0'?>
 <robot xmlns:xacro="http://www.ros.org/wiki/xacro" name="panda">
-  <xacro:macro name="panda_arm" params="arm_id:='panda' description_pkg:='aescape_panda_simulator' connected_to:='' in_gazebo='false' xyz:='0 0 0' rpy:='0 0 0'">
+  <xacro:macro name="panda_arm" params="arm_id:='panda' description_pkg:='aescape_gazebo' connected_to:='' in_gazebo='false' xyz:='0 0 0' rpy:='0 0 0'">
     <xacro:unless value="${not connected_to}">
       <joint name="${arm_id}_joint_${connected_to}" type="fixed">

File: urdf/robot.urdf.xacro (robot description, xacro)
@@ -2,5 +2,5 @@
 <robot xmlns:xacro="http://www.ros.org/wiki/xacro" name="aescape_robot">
   <!-- <xacro:include filename="$(find franka_description)/robots/panda_arm.xacro"/> -->
-  <xacro:include filename="$(find aescape_panda_simulator)/urdf/panda_arm.xacro"/>
+  <xacro:include filename="$(find aescape_gazebo)/urdf/panda_arm.xacro"/>
   <xacro:arg name="use_gazebo" default="true"/>
   <xacro:macro name="arm" params="arm_id:='panda' use_gazebo:='true'">
@@ -12,10 +12,10 @@
       <visual>
         <geometry>
-          <mesh filename="package://aescape_panda_simulator/meshes/visual/tool.dae" scale="0.019 0.019 0.019"/>>
+          <mesh filename="package://aescape_gazebo/meshes/visual/tool.dae" scale="0.019 0.019 0.019"/>>
         </geometry>
       </visual>
       <collision>
         <geometry>
-          <mesh filename="package://aescape_panda_simulator/meshes/collision/tool.stl" scale="0.019 0.019 0.019"/>
+          <mesh filename="package://aescape_gazebo/meshes/collision/tool.stl" scale="0.019 0.019 0.019"/>
         </geometry>
       </collision>
@@ -43,6 +43,6 @@
   <xacro:tool arm_id="left" rpy="${pi/2} 0 0"/-->
   <xacro:if value="$(arg use_gazebo)">
-    <xacro:include filename="$(find aescape_panda_simulator)/urdf/panda.gazebo.xacro"/>
-    <xacro:include filename="$(find aescape_panda_simulator)/urdf/panda.transmission.xacro"/>
+    <xacro:include filename="$(find aescape_gazebo)/urdf/panda.gazebo.xacro"/>
+    <xacro:include filename="$(find aescape_gazebo)/urdf/panda.transmission.xacro"/>
     <xacro:panda_gazebo robot_name="left_arm"/>
     <xacro:panda_gazebo robot_name="right_arm"/>
@@ -70,9 +70,4 @@
         <inertia ixx="1.0" ixy="0.0" ixz="0.0" iyy="1.0" iyz="0.0" izz="1.0"/>
     </inertial>
-    <!--gazebo reference="${robot_name}_link0">
-      <material>Gazebo/Grey</material>
-      <mu1>0.2</mu1>
-      <mu2>0.2</mu2>
-    </gazebo-->
   </link>
   <joint name="table_center_calibration" type="floating">
