Commit message: feat: dual robot launch file (gazebo, joint_state_controller and cartisian_motion_controller)

File: urdf/panda.transmission.xacro (robot description, xacro)
@@ -15,5 +15,5 @@
                 <robotNamespace>/${robot_name}</robotNamespace>
                 <updateRate>100.0</updateRate>
-                <topicName>ft_sensor_joint7</topicName>
+                <topicName>transformed_world</topicName>
                 <jointName>${robot_name}_joint7</jointName>
             </plugin>

File: urdf/panda_arm.xacro (robot description, xacro)
@@ -1,5 +1,5 @@
 <?xml version='1.0'?>
 <robot xmlns:xacro="http://www.ros.org/wiki/xacro" name="panda">
-  <xacro:macro name="panda_arm" params="arm_id:='panda' description_pkg:='aescape_panda_simulator' connected_to:=''  in_gazebo='false' xyz:='0 0 0' rpy:='0 0 0'">
+  <xacro:macro name="panda_arm" params="arm_id:='panda' description_pkg:='aescape_panda_simulator' connected_to:='' in_gazebo='false' xyz:='0 0 0' rpy:='0 0 0'">
     <xacro:unless value="${not connected_to}">
       <joint name="${arm_id}_joint_${connected_to}" type="fixed">
@@ -15,5 +15,5 @@
         <parent link="world" />
         <child link="${arm_id}_link0" />
-        <origin xyz="0.0 0.0 0.0" rpy="0.0 0.0 0.0" />
+        <origin rpy="${rpy}" xyz="${xyz}"/>
         <dynamics damping="${joint_damping}"/>
       </joint>

Commit message: feat: namespace and robot link and joint namez fixed

File: urdf/panda.transmission.xacro (robot description, xacro)
@@ -1,9 +1,9 @@
 <?xml version="1.0"?>
 <robot xmlns:xacro="http://www.ros.org/wiki/xacro">
-    <xacro:macro name="panda_transmission" params="robot_name">
+    <xacro:macro name="panda_transmission" params="robot_name robot_ns">
         <!-- Load ros control plugin -->
         <gazebo>
             <plugin name="gazebo_ros_control" filename="libgazebo_ros_control.so">
-                <robotNamespace>/${robot_name}</robotNamespace>
+                <robotNamespace>/${robot_ns}</robotNamespace>
                 <robotSimType>gazebo_ros_control/DefaultRobotHWSim</robotSimType>
                 <legacyModeNS>true</legacyModeNS>
@@ -13,5 +13,5 @@
         <gazebo>
             <plugin name="ft_sensor" filename="libgazebo_ros_ft_sensor.so">
-                <robotNamespace>/${robot_name}</robotNamespace>
+                <robotNamespace>/${robot_ns}</robotNamespace>
                 <updateRate>100.0</updateRate>
                 <topicName>transformed_world</topicName>

File: urdf/panda_arm.urdf.xacro (robot description, xacro)
@@ -2,4 +2,5 @@
 <robot xmlns:xacro="http://www.ros.org/wiki/xacro" name="panda">
   <xacro:arg name="robot_name" default="panda"/>
+  <xacro:arg name="robot_ns" default="panda"/>
   <xacro:arg name="load_gazebo" default="false"/>
   <xacro:arg name="origin_y" default="0.0"/>
@@ -10,11 +11,9 @@
   </xacro:unless>
   <xacro:if value="$(arg load_gazebo)">
+    <xacro:include filename="$(find aescape_gazebo)/urdf/panda.gazebo.xacro"/>
+    <xacro:include filename="$(find aescape_gazebo)/urdf/panda.transmission.xacro"/>
     <xacro:panda_arm in_gazebo="true" connected_to="world" arm_id="$(arg robot_name)" xyz="0.0 $(arg origin_y) 0.0"/>
-    <xacro:include filename="$(find aescape_gazebo)/urdf/panda.gazebo.xacro"/>
     <xacro:panda_gazebo robot_name="$(arg robot_name)"/>
-    <xacro:include filename="$(find aescape_gazebo)/urdf/panda.transmission.xacro"/>
-    <xacro:panda_transmission robot_name="$(arg robot_name)"/>
-    <xacro:include filename="$(find aescape_gazebo)/urdf/depth_camera.xacro"/>
-    <xacro:depth_camera camera_name="$(arg robot_name)" connected_to="world" xyz="1.0 $(arg origin_y) 1.0" rpy="0.0 0.7854 3.1416"/>
+    <xacro:panda_transmission robot_name="$(arg robot_name)" robot_ns="$(arg robot_ns)"/>
   </xacro:if>
 </robot>

File: urdf/robot.urdf.xacro (robot description, xacro)
@@ -5,9 +5,9 @@
   <xacro:arg name="use_gazebo" default="true"/>
   <xacro:macro name="arm" params="arm_id:='panda' use_gazebo:='true'">
-    <link name="${arm_id}_base_link"/>
-    <xacro:panda_arm arm_id="${arm_id}" connected_to="${arm_id}_base_link" in_gazebo="${use_gazebo}"  xyz="0 0 0" rpy="0 0 0"/>
+    <link name="${arm_id}_arm_base_link"/>
+    <xacro:panda_arm arm_id="${arm_id}_arm" connected_to="${arm_id}_arm_base_link" in_gazebo="${use_gazebo}"  xyz="0 0 0" rpy="0 0 0"/>
   </xacro:macro>
   <xacro:macro name="tool" params="rpy:='${pi/2} 0 0' arm_id:='panda'">
-      <link name="${arm_id}_tool_link">
+      <link name="${arm_id}_arm_tool_link">
       <visual>
         <geometry>
@@ -26,14 +26,14 @@
       </inertial>
     </link>
-    <joint name="${arm_id}_tool_joint" type="fixed">
+    <joint name="${arm_id}_arm_tool_joint" type="fixed">
       <origin rpy="${rpy}" xyz="-0.02 0.0 0.046"/>
-      <parent link="${arm_id}_link8"/>
-      <child link="${arm_id}_tool_link"/>
+      <parent link="${arm_id}_arm_link8"/>
+      <child link="${arm_id}_arm_tool_link"/>
       <axis xyz="0 0 1"/>
     </joint>
   </xacro:macro>
-  <joint name="right_base_link_calibration" type="fixed">
-    <parent link="left_base_link"/>
-    <child link="right_base_link"/>
+  <joint name="right_arm_base_link_calibration" type="fixed">
+    <parent link="left_arm_base_link"/>
+    <child link="right_arm_base_link"/>
     <origin xyz="1.0176 0.0111 -0.0046" rpy="0 0 ${pi}" /> <!-- Default Values -->
   </joint>
@@ -45,8 +45,8 @@
     <xacro:include filename="$(find aescape_gazebo)/urdf/panda.gazebo.xacro"/>
     <xacro:include filename="$(find aescape_gazebo)/urdf/panda.transmission.xacro"/>
-    <xacro:panda_gazebo robot_name="left"/>
-    <xacro:panda_gazebo robot_name="right"/>
-    <xacro:panda_transmission robot_name="left"/>
-    <xacro:panda_transmission robot_name="right"/>
+    <xacro:panda_gazebo robot_name="left_arm"/>
+    <xacro:panda_gazebo robot_name="right_arm"/>
+    <xacro:panda_transmission robot_name="left_arm" robot_ns="left"/>
+    <xacro:panda_transmission robot_name="right_arm" robot_ns="right"/>
   </xacro:if>
   <link name="table_center">
@@ -70,7 +70,12 @@
         <inertia ixx="1.0" ixy="0.0" ixz="0.0" iyy="1.0" iyz="0.0" izz="1.0"/>
     </inertial>
+    <!--gazebo reference="${robot_name}_link0">
+      <material>Gazebo/Grey</material>
+      <mu1>0.2</mu1>
+      <mu2>0.2</mu2>
+    </gazebo-->
   </link>
   <joint name="table_center_calibration" type="floating">
-    <parent link="left_base_link"/>
+    <parent link="left_arm_base_link"/>
     <child link="table_center"/>
     <origin xyz="0.5058 -0.023642 0.3334" rpy="0 0 0" /> <!-- Default Values -->
