Commit message: feat: cartesian_markers and cartesian_publisher launch file done

File: urdf/panda_arm.xacro (robot description, xacro)
@@ -239,10 +239,10 @@
       <visual>
         <geometry>
-          <mesh filename="package://${description_pkg}/meshes/visual/tool2.dae" scale="0.5 0.5 0.5"/>
-        </geometry>
-      </visual>
-      <collision>
-        <geometry>
-          <mesh filename="package://${description_pkg}/meshes/collision/tool2.stl" scale="0.5 0.5 0.5"/>
+          <mesh filename="package://${description_pkg}/meshes/visual/tool.dae" scale="0.019 0.019 0.019"/>
+        </geometry>
+      </visual>
+      <collision>
+        <geometry>
+          <mesh filename="package://${description_pkg}/meshes/collision/tool.stl" scale="0.019 0.019 0.019"/>
         </geometry>
       </collision>
@@ -255,5 +255,6 @@
     <!-- Joint8 -->
     <joint name="joint8" type="fixed">
-      <origin rpy="${pi/2} 0 0" xyz="-0.40 -0.654 -0.6195"/>
+      <!--origin rpy="${pi/2} 0 0" xyz="-0.40 -0.654 -0.6195"/-->
+      <origin rpy="${pi/2} 0 0" xyz="-0.02 0.0 0.046"/>
       <parent link="link7"/>
       <child link="link8"/>

Commit message: fix: robot.urdf.xacro fixed

File: urdf/panda_arm.xacro (robot description, xacro)
@@ -220,5 +220,5 @@
       <dynamics damping="1.0" friction="0.5"/>
     </joint>
-    <link name="${arm_id}_link8">
+    <!--link name="${arm_id}_link8">
       <visual>
         <geometry>
@@ -242,4 +242,17 @@
       <child link="${arm_id}_link8"/>
       <axis xyz="0 0 1"/>
+    </joint-->
+    <link name="${arm_id}_link8">
+      <inertial>
+        <origin rpy="0 0 0" xyz="0 0 0"/>
+        <mass value="0.0"/>
+        <inertia ixx="0.001" ixy="0.0" ixz="0.0" iyy="0.001" iyz="0.0" izz="0.001"/>
+      </inertial>
+    </link>
+    <joint name="${arm_id}_joint8" type="fixed">
+      <origin rpy="0 0 0" xyz="0 0 0"/>
+      <parent link="${arm_id}_link7"/>
+      <child link="${arm_id}_link8"/>
+      <axis xyz="0 0 0"/>
     </joint>
   </xacro:macro>

File: urdf/robot.urdf.xacro (robot description, xacro)
@@ -4,32 +4,37 @@
   <xacro:include filename="$(find aescape_gazebo)/urdf/panda_arm.xacro"/>
   <xacro:arg name="use_gazebo" default="true"/>
+  <xacro:arg name="load_tool" default="false"/>
   <xacro:macro name="arm" params="arm_id:='panda' use_gazebo:='true'">
     <link name="${arm_id}_arm_base_link"/>
     <xacro:panda_arm arm_id="${arm_id}_arm" connected_to="${arm_id}_arm_base_link" in_gazebo="${use_gazebo}"  xyz="0 0 0" rpy="0 0 0"/>
   </xacro:macro>
-  <xacro:macro name="tool" params="rpy:='${pi/2} 0 0' arm_id:='panda'">
-      <link name="${arm_id}_arm_tool_link">
+  <xacro:macro name="tool" params="rpy:='${pi/2} 0 0' xyz:='0 0 0' arm_id:='panda'">
+    <link name="${arm_id}_arm_tool_link">
       <visual>
         <geometry>
-          <mesh filename="package://aescape_gazebo/meshes/visual/tool.dae" scale="0.019 0.019 0.019"/>>
+          <mesh filename="package://aescape_gazebo/meshes/visual/tool.dae" scale="0.019 0.019 0.019"/>
         </geometry>
       </visual>
       <collision>
         <geometry>
-          <mesh filename="package://aescape_gazebo/meshes/collision/tool.stl" scale="0.019 0.019 0.019"/>
+          <mesh filename="package://aescape_gazebo/meshes/visual/tool.stl" scale="0.019 0.019 0.019"/>
         </geometry>
       </collision>
       <inertial>
         <origin xyz="0 0 0" rpy="0 0 0"/>
-        <mass value="0.0"/>
-        <inertia ixx="0.001" ixy="0.0" ixz="0.0" iyy="0.001" iyz="0.0" izz="0.001"/>
+        <mass value="0.68"/>
+        <inertia ixx="0.1" ixy="0.0" ixz="0.0" iyy="0.1" iyz="0.0" izz="0.1"/>
       </inertial>
     </link>
-    <joint name="${arm_id}_arm_tool_joint" type="fixed">
-      <origin rpy="${rpy}" xyz="-0.02 0.0 0.046"/>
+    <joint name="${arm_id}_arm_joint_tool" type="fixed">
       <parent link="${arm_id}_arm_link8"/>
       <child link="${arm_id}_arm_tool_link"/>
-      <axis xyz="0 0 1"/>
+      <origin rpy="${rpy}" xyz="${xyz}"/>
     </joint>
+    <gazebo reference="${arm_id}_arm_tool_link">
+      <material>Gazebo/Grey</material>
+      <mu1>0.2</mu1>
+      <mu2>0.2</mu2>
+    </gazebo>
   </xacro:macro>
   <joint name="right_arm_base_link_calibration" type="fixed">
@@ -40,6 +45,6 @@
   <xacro:arm arm_id="right"/>
   <xacro:arm arm_id="left"/>
-  <!--xacro:tool arm_id="right" rpy="${pi/2} 0 ${pi}"/>
-  <xacro:tool arm_id="left" rpy="${pi/2} 0 0"/-->
+  <xacro:tool arm_id="left"  rpy="${pi/2} 0 0" xyz="-0.02 0.0 0.046"/>
+  <xacro:tool arm_id="right" rpy="${pi/2} 0 0" xyz="-0.02 0.0 0.046"/>
   <xacro:if value="$(arg use_gazebo)">
     <xacro:include filename="$(find aescape_gazebo)/urdf/panda.gazebo.xacro"/>
