Commit message: fix: left_tp.stl fixed

File: urdf/tool.xacro (robot description, xacro)
@@ -10,5 +10,5 @@
       <collision>
         <geometry>
-          <mesh filename="package://aescape_gazebo/meshes/visual/left_tp.stl"/>
+          <mesh filename="package://aescape_gazebo/meshes/collision/left_tp.stl"/>
         </geometry>
       </collision>

Commit message: feat: bumper sensor added

File: urdf/tool.xacro (robot description, xacro)
@@ -28,4 +28,14 @@
       <mu1>0.2</mu1>
       <mu2>0.2</mu2>
+      <sensor name="${arm_id}_arm_tool_bumper" type="contact">
+        <always_on>true</always_on>
+        <contact>
+          <collision>${arm_id}_arm_link7_fixed_joint_lump__${arm_id}_arm_tool_link_collision_1</collision>
+        </contact>
+        <plugin name="${arm_id}_arm_tool_plugin" filename="libgazebo_ros_bumper.so">
+          <bumperTopicName>/${arm_id}/${arm_id}_arm_tool_link/bumper</bumperTopicName>
+          <frameName>${arm_id}_arm_tool_link</frameName>
+        </plugin>
+      </sensor>
     </gazebo>
   </xacro:macro>
