Commit message: feat: arm_id added to all joints and links

File: urdf/panda.gazebo.xacro (robot description, xacro)
@@ -1,7 +1,6 @@
 <?xml version="1.0"?>
 <robot xmlns:xacro="http://www.ros.org/wiki/xacro">
-    <xacro:macro name="panda_gazebo">
-        <!-- Link0 -->
-        <gazebo reference="link0">
+    <xacro:macro name="panda_gazebo" params="robot_name">
+        <gazebo reference="${robot_name}_link0">
             <material>Gazebo/Grey</material>
             <mu1>0.2</mu1>
@@ -9,5 +8,5 @@
         </gazebo>
         <!-- Link1 -->
-        <gazebo reference="link1">
+        <gazebo reference="${robot_name}_link1">
             <material>Gazebo/White</material>
             <mu1>0.2</mu1>
@@ -15,5 +14,5 @@
         </gazebo>
         <!-- Link2 -->
-        <gazebo reference="link2">
+        <gazebo reference="${robot_name}_link2">
             <material>Gazebo/White</material>
             <mu1>0.2</mu1>
@@ -21,5 +20,5 @@
         </gazebo>
         <!-- Link3 -->
-        <gazebo reference="link3">
+        <gazebo reference="${robot_name}_link3">
             <material>Gazebo/White</material>
             <mu1>0.2</mu1>
@@ -27,5 +26,5 @@
         </gazebo>
         <!-- Link4 -->
-        <gazebo reference="link4">
+        <gazebo reference="${robot_name}_link4">
             <material>Gazebo/White</material>
             <mu1>0.2</mu1>
@@ -33,5 +32,5 @@
         </gazebo>
         <!-- Link5 -->
-        <gazebo reference="link5">
+        <gazebo reference="${robot_name}_link5">
             <material>Gazebo/White</material>
             <mu1>0.2</mu1>
@@ -39,5 +38,5 @@
         </gazebo>
         <!-- Link6 -->
-        <gazebo reference="link6">
+        <gazebo reference="${robot_name}_link6">
             <material>Gazebo/White</material>
             <mu1>0.2</mu1>
@@ -45,52 +44,52 @@
         </gazebo>
         <!-- Link7 -->
-        <gazebo reference="link7">
-            <material>Gazebo/White</material>
+        <gazebo reference="${robot_name}_link7">
+            <material>Gazebo/Grey</material>
             <mu1>0.2</mu1>
             <mu2>0.2</mu2>
         </gazebo>
         <!-- Link8 -->
-        <gazebo reference="link8">
-            <material>Gazebo/White</material>
+        <gazebo reference="${robot_name}_link8">
+            <material>Gazebo/Grey</material>
             <mu1>0.2</mu1>
             <mu2>0.2</mu2>
         </gazebo>
         <!-- Joint1 -->
-        <gazebo reference="joint1">
+        <gazebo reference="${robot_name}_joint1">
           <implicitSpringDamper>1</implicitSpringDamper>
           <provideFeedback>true</provideFeedback>
         </gazebo>
         <!-- Joint2 -->
-        <gazebo reference="joint2">
+        <gazebo reference="${robot_name}_joint2">
           <implicitSpringDamper>1</implicitSpringDamper>
           <provideFeedback>true</provideFeedback>
         </gazebo>
         <!-- Joint3 -->
-        <gazebo reference="joint3">
+        <gazebo reference="${robot_name}_joint3">
           <implicitSpringDamper>1</implicitSpringDamper>
           <provideFeedback>true</provideFeedback>
         </gazebo>
         <!-- Joint4 -->
-        <gazebo reference="joint4">
+        <gazebo reference="${robot_name}_joint4">
           <implicitSpringDamper>1</implicitSpringDamper>
           <provideFeedback>true</provideFeedback>
         </gazebo>
         <!-- Joint5 -->
-        <gazebo reference="joint5">
+        <gazebo reference="${robot_name}_joint5">
+          <implicitSpringDamper>1</implicitSpringDamper>
+          <provideFeedback>true</provideFeedback>
+        </gazebo>
+        <!-- Joint5 -->
+        <gazebo reference="${robot_name}_joint6">
           <implicitSpringDamper>1</implicitSpringDamper>
           <provideFeedback>true</provideFeedback>
         </gazebo>
         <!-- Joint6 -->
-        <gazebo reference="joint6">
+        <gazebo reference="${robot_name}_joint7">
           <implicitSpringDamper>1</implicitSpringDamper>
           <provideFeedback>true</provideFeedback>
         </gazebo>
         <!-- Joint7 -->
-        <gazebo reference="joint7">
-          <implicitSpringDamper>1</implicitSpringDamper>
-          <provideFeedback>true</provideFeedback>
-        </gazebo>
-        <!-- Joint8 -->
-        <gazebo reference="joint8">
+        <gazebo reference="${robot_name}_joint8">
           <implicitSpringDamper>1</implicitSpringDamper>
           <provideFeedback>true</provideFeedback>

File: urdf/panda.transmission.xacro (robot description, xacro)
@@ -1,9 +1,9 @@
 <?xml version="1.0"?>
 <robot xmlns:xacro="http://www.ros.org/wiki/xacro">
-    <xacro:macro name="panda_transmission">
+    <xacro:macro name="panda_transmission" params="robot_name">
         <!-- Load ros control plugin -->
         <gazebo>
             <plugin name="gazebo_ros_control" filename="libgazebo_ros_control.so">
-                <robotNamespace>/panda</robotNamespace>
+                <robotNamespace>/${robot_name}</robotNamespace>
                 <robotSimType>gazebo_ros_control/DefaultRobotHWSim</robotSimType>
                 <legacyModeNS>true</legacyModeNS>
@@ -13,83 +13,76 @@
         <gazebo>
             <plugin name="ft_sensor" filename="libgazebo_ros_ft_sensor.so">
-                <robotNamespace>/panda</robotNamespace>
+                <robotNamespace>/${robot_name}</robotNamespace>
                 <updateRate>100.0</updateRate>
                 <topicName>ft_sensor_joint7</topicName>
-                <jointName>joint7</jointName>
+                <jointName>${robot_name}_joint7</jointName>
             </plugin>
         </gazebo>
-        <!-- Transmission1 -->
-        <transmission name="transmision1">
+                <transmission name="${robot_name}_tran_1">
             <type>transmission_interface/SimpleTransmission</type>
-            <joint name="joint1">
+            <joint name="${robot_name}_joint1">
                 <hardwareInterface>hardware_interface/PositionJointInterface</hardwareInterface>
             </joint>
-            <actuator name="motor1">
+            <actuator name="${robot_name}_motor_1">
                 <hardwareInterface>hardware_interface/PositionJointInterface</hardwareInterface>
                 <mechanicalReduction>1</mechanicalReduction>
             </actuator>
         </transmission>
-        <!-- Transmission2 -->
-        <transmission name="transmision2">
+        <transmission name="${robot_name}_tran_2">
             <type>transmission_interface/SimpleTransmission</type>
-            <joint name="joint2">
+            <joint name="${robot_name}_joint2">
                 <hardwareInterface>hardware_interface/PositionJointInterface</hardwareInterface>
             </joint>
-            <actuator name="motor2">
+            <actuator name="${robot_name}_motor_2">
                 <hardwareInterface>hardware_interface/PositionJointInterface</hardwareInterface>
                 <mechanicalReduction>1</mechanicalReduction>
             </actuator>
         </transmission>
-        <!-- Transmission3 -->
-        <transmission name="transmision3">
+        <transmission name="${robot_name}_tran_3">
             <type>transmission_interface/SimpleTransmission</type>
-            <joint name="joint3">
+            <joint name="${robot_name}_joint3">
                 <hardwareInterface>hardware_interface/PositionJointInterface</hardwareInterface>
             </joint>
-            <actuator name="motor3">
+            <actuator name="${robot_name}_motor_3">
                 <hardwareInterface>hardware_interface/PositionJointInterface</hardwareInterface>
                 <mechanicalReduction>1</mechanicalReduction>
             </actuator>
         </transmission>
-        <!-- Transmission4 -->
-        <transmission name="transmision4">
+        <transmission name="${robot_name}_tran_4">
             <type>transmission_interface/SimpleTransmission</type>
-            <joint name="joint4">
+            <joint name="${robot_name}_joint4">
                 <hardwareInterface>hardware_interface/PositionJointInterface</hardwareInterface>
             </joint>
-            <actuator name="motor4">
+            <actuator name="${robot_name}_motor_4">
                 <hardwareInterface>hardware_interface/PositionJointInterface</hardwareInterface>
                 <mechanicalReduction>1</mechanicalReduction>
             </actuator>
         </transmission>
-        <!-- Transmission5 -->
-        <transmission name="transmision5">
+        <transmission name="${robot_name}_tran_5">
             <type>transmission_interface/SimpleTransmission</type>
-            <joint name="joint5">
+            <joint name="${robot_name}_joint5">
                 <hardwareInterface>hardware_interface/PositionJointInterface</hardwareInterface>
             </joint>
-            <actuator name="motor5">
+            <actuator name="${robot_name}_motor_5">
                 <hardwareInterface>hardware_interface/PositionJointInterface</hardwareInterface>
                 <mechanicalReduction>1</mechanicalReduction>
             </actuator>
         </transmission>
-        <!-- Transmission6 -->
-        <transmission name="transmision6">
+        <transmission name="${robot_name}_tran_6">
             <type>transmission_interface/SimpleTransmission</type>
-            <joint name="joint6">
+            <joint name="${robot_name}_joint6">
                 <hardwareInterface>hardware_interface/PositionJointInterface</hardwareInterface>
             </joint>
-            <actuator name="motor6">
+            <actuator name="${robot_name}_motor_6">
                 <hardwareInterface>hardware_interface/PositionJointInterface</hardwareInterface>
                 <mechanicalReduction>1</mechanicalReduction>
             </actuator>
         </transmission>
-        <!-- Transmission7 -->
-        <transmission name="transmision7">
+        <transmission name="${robot_name}_tran_7">
             <type>transmission_interface/SimpleTransmission</type>
-            <joint name="joint7">
+            <joint name="${robot_name}_joint7">
                 <hardwareInterface>hardware_interface/PositionJointInterface</hardwareInterface>
             </joint>
-            <actuator name="motor7">
+            <actuator name="${robot_name}_motor_7">
                 <hardwareInterface>hardware_interface/PositionJointInterface</hardwareInterface>
                 <mechanicalReduction>1</mechanicalReduction>

File: urdf/panda_arm.urdf.xacro (robot description, xacro)
@@ -1,15 +1,16 @@
 <?xml version="1.0"?>
 <robot xmlns:xacro="http://www.ros.org/wiki/xacro" name="panda">
+  <xacro:arg name="robot_name" default="panda"/>
   <xacro:arg name="load_gazebo" default="false"/>
   <xacro:include filename="$(find aescape_panda_simulator)/urdf/panda_arm.xacro"/>
   <xacro:unless value="$(arg load_gazebo)">
-    <xacro:panda_arm />
+    <xacro:panda_arm arm_id="$(arg robot_name)"/>
   </xacro:unless>
   <xacro:if value="$(arg load_gazebo)">
-    <xacro:panda_arm in_gazebo="true"/>
+    <xacro:panda_arm in_gazebo="true" arm_id="$(arg robot_name)"/>
     <xacro:include filename="$(find aescape_panda_simulator)/urdf/panda.gazebo.xacro"/>
-    <xacro:panda_gazebo/>
+    <xacro:panda_gazebo robot_name="$(arg robot_name)"/>
     <xacro:include filename="$(find aescape_panda_simulator)/urdf/panda.transmission.xacro"/>
-    <xacro:panda_transmission/>
+    <xacro:panda_transmission robot_name="$(arg robot_name)"/>
   </xacro:if>
 </robot>

File: urdf/panda_arm.xacro (robot description, xacro)
@@ -3,7 +3,7 @@
   <xacro:macro name="panda_arm" params="arm_id:='panda' description_pkg:='aescape_panda_simulator' connected_to:=''  in_gazebo='false' xyz:='0 0 0' rpy:='0 0 0'">
     <xacro:unless value="${not connected_to}">
-      <joint name="joint_${connected_to}" type="fixed">
+      <joint name="${arm_id}_joint_${connected_to}" type="fixed">
         <parent link="${connected_to}"/>
-        <child link="link0"/>
+        <child link="${arm_id}_link0"/>
         <origin rpy="${rpy}" xyz="${xyz}"/>
       </joint>
@@ -14,11 +14,10 @@
       <joint name="robot_to_world" type="fixed">
         <parent link="world" />
-        <child link="link0" />
+        <child link="${arm_id}_link0" />
         <origin xyz="0.0 0.0 0.0" rpy="0.0 0.0 0.0" />
         <dynamics damping="${joint_damping}"/>
       </joint>
     </xacro:unless>
-    <!-- Link0 -->
-    <link name="link0">
+    <link name="${arm_id}_link0">
       <visual>
         <geometry>
@@ -39,6 +38,5 @@
       </xacro:unless>
     </link>
-    <!-- Link1 -->
-    <link name="link1">
+    <link name="${arm_id}_link1">
       <visual>
         <geometry>
@@ -57,16 +55,14 @@
       </inertial>
     </link>
-    <!-- Joint1 -->
-    <joint name="joint1" type="revolute">
+    <joint name="${arm_id}_joint1" type="revolute">
       <safety_controller k_position="100.0" k_velocity="40.0" soft_lower_limit="-2.8973" soft_upper_limit="2.8973"/>
       <origin rpy="0 0 0" xyz="0 0 0.333"/>
-      <parent link="link0"/>
-      <child link="link1"/>
+      <parent link="${arm_id}_link0"/>
+      <child link="${arm_id}_link1"/>
       <axis xyz="0 0 1"/>
       <limit effort="87" lower="-2.8973" upper="2.8973" velocity="2.1750"/>
       <dynamics damping="10.0" friction="5.0"/>
     </joint>
-    <!-- Link2 -->
-    <link name="link2">
+    <link name="${arm_id}_link2">
       <visual>
         <geometry>
@@ -85,16 +81,14 @@
       </inertial>
     </link>
-    <!-- Joint2 -->
-    <joint name="joint2" type="revolute">
+    <joint name="${arm_id}_joint2" type="revolute">
       <safety_controller k_position="100.0" k_velocity="40.0" soft_lower_limit="-1.7628" soft_upper_limit="1.7628"/>
       <origin rpy="${-pi/2} 0 0" xyz="0 0 0"/>
-      <parent link="link1"/>
-      <child link="link2"/>
+      <parent link="${arm_id}_link1"/>
+      <child link="${arm_id}_link2"/>
       <axis xyz="0 0 1"/>
       <limit effort="87" lower="-1.7628" upper="1.7628" velocity="2.1750"/>
       <dynamics damping="5.0" friction="2.0"/>
     </joint>
-    <!-- Link3 -->
-    <link name="link3">
+    <link name="${arm_id}_link3">
       <visual>
         <geometry>
@@ -113,16 +107,14 @@
       </inertial>
     </link>
-    <!-- Joint3 -->
-    <joint name="joint3" type="revolute">
+    <joint name="${arm_id}_joint3" type="revolute">
       <safety_controller k_position="100.0" k_velocity="40.0" soft_lower_limit="-2.8973" soft_upper_limit="2.8973"/>
       <origin rpy="${pi/2} 0 0" xyz="0 -0.316 0"/>
-      <parent link="link2"/>
-      <child link="link3"/>
+      <parent link="${arm_id}_link2"/>
+      <child link="${arm_id}_link3"/>
       <axis xyz="0 0 1"/>
       <limit effort="87" lower="-2.8973" upper="2.8973" velocity="2.1750"/>
       <dynamics damping="5.0" friction="2.0"/>
     </joint>
-    <!-- Link4 -->
-    <link name="link4">
+    <link name="${arm_id}_link4">
       <visual>
         <geometry>
@@ -141,16 +133,14 @@
       </inertial>
     </link>
-    <!-- Joint4 -->
-    <joint name="joint4" type="revolute">
+    <joint name="${arm_id}_joint4" type="revolute">
       <safety_controller k_position="100.0" k_velocity="40.0" soft_lower_limit="-3.0718" soft_upper_limit="-0.0698"/>
       <origin rpy="${pi/2} 0 0" xyz="0.0825 0 0"/>
-      <parent link="link3"/>
-      <child link="link4"/>
+      <parent link="${arm_id}_link3"/>
+      <child link="${arm_id}_link4"/>
       <axis xyz="0 0 1"/>
       <limit effort="87" lower="-3.0718" upper="-0.0698" velocity="2.1750"/>
       <dynamics damping="1.0" friction="0.5"/>
     </joint>
-    <!-- Link5 -->
-    <link name="link5">
+    <link name="${arm_id}_link5">
       <visual>
         <geometry>
@@ -169,16 +159,14 @@
       </inertial>
     </link>
-    <!-- Joint5 -->
-    <joint name="joint5" type="revolute">
+    <joint name="${arm_id}_joint5" type="revolute">
       <safety_controller k_position="100.0" k_velocity="40.0" soft_lower_limit="-2.8973" soft_upper_limit="2.8973"/>
       <origin rpy="${-pi/2} 0 0" xyz="-0.0825 0.384 0"/>
-      <parent link="link4"/>
-      <child link="link5"/>
+      <parent link="${arm_id}_link4"/>
+      <child link="${arm_id}_link5"/>
       <axis xyz="0 0 1"/>
       <limit effort="12" lower="-2.8973" upper="2.8973" velocity="2.6100"/>
       <dynamics damping="2.0" friction="1.0"/>
     </joint>
-    <!-- Link6 -->
-    <link name="link6">
+    <link name="${arm_id}_link6">
       <visual>
         <geometry>
@@ -197,16 +185,14 @@
       </inertial>
     </link>
-    <!-- Joint6 -->
-    <joint name="joint6" type="revolute">
+    <joint name="${arm_id}_joint6" type="revolute">
       <safety_controller k_position="100.0" k_velocity="40.0" soft_lower_limit="-0.0175" soft_upper_limit="3.7525"/>
       <origin rpy="${pi/2} 0 0" xyz="0 0 0"/>
-      <parent link="link5"/>
-      <child link="link6"/>
+      <parent link="${arm_id}_link5"/>
+      <child link="${arm_id}_link6"/>
       <axis xyz="0 0 1"/>
       <limit effort="12" lower="-0.0175" upper="3.7525" velocity="2.6100"/>
       <dynamics damping="1.0" friction="0.5"/>
     </joint>
-    <!-- Link7 -->
-    <link name="link7">
+    <link name="${arm_id}_link7">
       <visual>
         <geometry>
@@ -225,19 +211,17 @@
       </inertial>
     </link>
-    <!-- Joint7 -->
-    <joint name="joint7" type="revolute">
+    <joint name="${arm_id}_joint7" type="revolute">
       <safety_controller k_position="100.0" k_velocity="40.0" soft_lower_limit="-2.8973" soft_upper_limit="2.8973"/>
       <origin rpy="${pi/2} 0 0" xyz="0.088 -0.106 0.0"/>
-      <parent link="link6"/>
-      <child link="link7"/>
+      <parent link="${arm_id}_link6"/>
+      <child link="${arm_id}_link7"/>
       <axis xyz="0 0 1"/>
       <limit effort="12" lower="-2.8973" upper="2.8973" velocity="2.6100"/>
       <dynamics damping="1.0" friction="0.5"/>
     </joint>
-    <!-- Link8 -->
-    <link name="link8">
-      <visual>
-        <geometry>
-          <mesh filename="package://${description_pkg}/meshes/visual/tool.dae" scale="0.019 0.019 0.019"/>
+    <link name="${arm_id}_link8">
+      <visual>
+        <geometry>
+          <mesh filename="package://${description_pkg}/meshes/visual/tool.dae" scale="0.019 0.019 0.019"/>>
         </geometry>
       </visual>
@@ -250,13 +234,11 @@
         <origin xyz="0 0 0" rpy="0 0 0"/>
         <mass value="0.0"/>
-        <inertia ixx="0.0" ixy="0.0" ixz="0.0" iyy="0.0" iyz="0.0" izz="0.0"/>
-      </inertial>
-    </link>
-    <!-- Joint8 -->
-    <joint name="joint8" type="fixed">
-      <!--origin rpy="${pi/2} 0 0" xyz="-0.40 -0.654 -0.6195"/-->
+        <inertia ixx="0.001" ixy="0.0" ixz="0.0" iyy="0.001" iyz="0.0" izz="0.001"/>
+      </inertial>
+    </link>
+    <joint name="${arm_id}_joint8" type="fixed">
       <origin rpy="${pi/2} 0 0" xyz="-0.02 0.0 0.046"/>
-      <parent link="link7"/>
-      <child link="link8"/>
+      <parent link="${arm_id}_link7"/>
+      <child link="${arm_id}_link8"/>
       <axis xyz="0 0 1"/>
     </joint>
