Commit message: feat: Robots renamed to left and right

File: urdf/robot.urdf.xacro (robot description, xacro)
@@ -5,9 +5,9 @@
   <xacro:arg name="use_gazebo" default="true"/>
   <xacro:macro name="arm" params="arm_id:='panda' use_gazebo:='true'">
-    <link name="${arm_id}_arm_base_link"/>
-    <xacro:panda_arm arm_id="${arm_id}_arm" connected_to="${arm_id}_arm_base_link" in_gazebo="${use_gazebo}"  xyz="0 0 0" rpy="0 0 0"/>
+    <link name="${arm_id}_base_link"/>
+    <xacro:panda_arm arm_id="${arm_id}" connected_to="${arm_id}_base_link" in_gazebo="${use_gazebo}"  xyz="0 0 0" rpy="0 0 0"/>
   </xacro:macro>
   <xacro:macro name="tool" params="rpy:='${pi/2} 0 0' arm_id:='panda'">
-      <link name="${arm_id}_arm_tool_link">
+      <link name="${arm_id}_tool_link">
       <visual>
         <geometry>
@@ -26,14 +26,14 @@
       </inertial>
     </link>
-    <joint name="${arm_id}_arm_tool_joint" type="fixed">
+    <joint name="${arm_id}_tool_joint" type="fixed">
       <origin rpy="${rpy}" xyz="-0.02 0.0 0.046"/>
-      <parent link="${arm_id}_arm_link8"/>
-      <child link="${arm_id}_arm_tool_link"/>
+      <parent link="${arm_id}_link8"/>
+      <child link="${arm_id}_tool_link"/>
       <axis xyz="0 0 1"/>
     </joint>
   </xacro:macro>
-  <joint name="right_arm_base_link_calibration" type="fixed">
-    <parent link="left_arm_base_link"/>
-    <child link="right_arm_base_link"/>
+  <joint name="right_base_link_calibration" type="fixed">
+    <parent link="left_base_link"/>
+    <child link="right_base_link"/>
     <origin xyz="1.0176 0.0111 -0.0046" rpy="0 0 ${pi}" /> <!-- Default Values -->
   </joint>
@@ -45,8 +45,8 @@
     <xacro:include filename="$(find aescape_gazebo)/urdf/panda.gazebo.xacro"/>
     <xacro:include filename="$(find aescape_gazebo)/urdf/panda.transmission.xacro"/>
-    <xacro:panda_gazebo robot_name="left_arm"/>
-    <xacro:panda_gazebo robot_name="right_arm"/>
-    <xacro:panda_transmission robot_name="left_arm"/>
-    <xacro:panda_transmission robot_name="right_arm"/>
+    <xacro:panda_gazebo robot_name="left"/>
+    <xacro:panda_gazebo robot_name="right"/>
+    <xacro:panda_transmission robot_name="left"/>
+    <xacro:panda_transmission robot_name="right"/>
   </xacro:if>
   <link name="table_center">
@@ -72,5 +72,5 @@
   </link>
   <joint name="table_center_calibration" type="floating">
-    <parent link="left_arm_base_link"/>
+    <parent link="left_base_link"/>
     <child link="table_center"/>
     <origin xyz="0.5058 -0.023642 0.3334" rpy="0 0 0" /> <!-- Default Values -->

Commit message: feat: tool xacro done, depth_cameras added

File: urdf/robot.urdf.xacro (robot description, xacro)
@@ -1,6 +1,6 @@
 <?xml version="1.0" encoding="utf-8"?>
 <robot xmlns:xacro="http://www.ros.org/wiki/xacro" name="aescape_robot">
-  <!-- <xacro:include filename="$(find franka_description)/robots/panda_arm.xacro"/> -->
   <xacro:include filename="$(find aescape_gazebo)/urdf/panda_arm.xacro"/>
+  <xacro:include filename="$(find aescape_gazebo)/urdf/tool.xacro"/>
   <xacro:arg name="use_gazebo" default="true"/>
   <xacro:arg name="load_tool" default="false"/>
@@ -8,33 +8,4 @@
     <link name="${arm_id}_arm_base_link"/>
     <xacro:panda_arm arm_id="${arm_id}_arm" connected_to="${arm_id}_arm_base_link" in_gazebo="${use_gazebo}"  xyz="0 0 0" rpy="0 0 0"/>
-  </xacro:macro>
-  <xacro:macro name="tool" params="rpy:='${pi/2} 0 0' xyz:='0 0 0' arm_id:='panda'">
-    <link name="${arm_id}_arm_tool_link">
-      <visual>
-        <geometry>
-          <mesh filename="package://aescape_gazebo/meshes/visual/tool.dae" scale="0.019 0.019 0.019"/>
-        </geometry>
-      </visual>
-      <collision>
-        <geometry>
-          <mesh filename="package://aescape_gazebo/meshes/visual/tool.stl" scale="0.019 0.019 0.019"/>
-        </geometry>
-      </collision>
-      <inertial>
-        <origin xyz="0 0 0" rpy="0 0 0"/>
-        <mass value="0.68"/>
-        <inertia ixx="0.1" ixy="0.0" ixz="0.0" iyy="0.1" iyz="0.0" izz="0.1"/>
-      </inertial>
-    </link>
-    <joint name="${arm_id}_arm_joint_tool" type="fixed">
-      <parent link="${arm_id}_arm_link8"/>
-      <child link="${arm_id}_arm_tool_link"/>
-      <origin rpy="${rpy}" xyz="${xyz}"/>
-    </joint>
-    <gazebo reference="${arm_id}_arm_tool_link">
-      <material>Gazebo/Grey</material>
-      <mu1>0.2</mu1>
-      <mu2>0.2</mu2>
-    </gazebo>
   </xacro:macro>
   <joint name="right_arm_base_link_calibration" type="fixed">
@@ -45,13 +16,17 @@
   <xacro:arm arm_id="right"/>
   <xacro:arm arm_id="left"/>
-  <xacro:tool arm_id="left"  rpy="${pi/2} 0 0" xyz="-0.02 0.0 0.046"/>
-  <xacro:tool arm_id="right" rpy="${pi/2} 0 0" xyz="-0.02 0.0 0.046"/>
+  <xacro:tool arm_id="left"  connected_to="left_arm_link8" rpy="${pi/2} 0 0" xyz="-0.02 0.0 0.046"/>
+  <xacro:tool arm_id="right" connected_to="right_arm_link8" rpy="${pi/2} 0 0" xyz="-0.02 0.0 0.046"/>
   <xacro:if value="$(arg use_gazebo)">
     <xacro:include filename="$(find aescape_gazebo)/urdf/panda.gazebo.xacro"/>
     <xacro:include filename="$(find aescape_gazebo)/urdf/panda.transmission.xacro"/>
+    <xacro:include filename="$(find aescape_gazebo)/urdf/depth_camera.xacro"/>
     <xacro:panda_gazebo robot_name="left_arm"/>
     <xacro:panda_gazebo robot_name="right_arm"/>
     <xacro:panda_transmission robot_name="left_arm" robot_ns="left"/>
     <xacro:panda_transmission robot_name="right_arm" robot_ns="right"/>
+    <xacro:depth_camera camera_name="left_camera_base" connected_to="left_arm_base_link" xyz="0.0 0.0 1.0" rpy="0.0 0.0 0.0"/>
+    <xacro:depth_camera camera_name="center_camera_base" connected_to="left_arm_base_link" xyz="0.0 -0.6 1.0" rpy="0.0 0.0 0.0"/>
+    <xacro:depth_camera camera_name="right_camera_base" connected_to="left_arm_base_link" xyz="0.0 -1.2 1.0" rpy="0.0 0.0 0.0"/>
   </xacro:if>
   <link name="table_center">
@@ -60,7 +35,7 @@
       	<box size="0.76 1.83 0.1"/>
       </geometry>
-      <material name="Grey">
+      <!--material name="Grey">
 	      <color rgba="0.5 0.5 0.5 0.8"/>
-      </material>
+      </material-->
       <origin rpy="0 0 0" xyz="0 -0.6332 -0.05"/>
     </visual>
@@ -75,11 +50,11 @@
         <inertia ixx="1.0" ixy="0.0" ixz="0.0" iyy="1.0" iyz="0.0" izz="1.0"/>
     </inertial>
-    <!--gazebo reference="${robot_name}_link0">
-      <material>Gazebo/Grey</material>
+    <gazebo reference="table_center">
+      <material>Gazebo/Black</material>
       <mu1>0.2</mu1>
       <mu2>0.2</mu2>
-    </gazebo-->
+    </gazebo>
   </link>
-  <joint name="table_center_calibration" type="floating">
+  <joint name="table_center_calibration" type="fixed">
     <parent link="left_arm_base_link"/>
     <child link="table_center"/>

File: urdf/tool.xacro (robot description, xacro)
@@ -1,30 +1,27 @@
 <?xml version="1.0" encoding="utf-8"?>
 <robot xmlns:xacro="http://www.ros.org/wiki/xacro" name="tool">
-  <xacro:macro name="tool" params="robot_ns:='' connected_to:='' in_gazebo='true' rpy:='0 0 0' xyz:='0 0 0' ">
+  <xacro:macro name="tool" params="arm_id:='panda' connected_to:='' rpy:='${pi/2} 0 0' xyz:='-0.02 0.0 0.046'">
     <link name="${arm_id}_arm_tool_link">
       <visual>
         <geometry>
-          <mesh filename="package://aescape_gazebo/meshes/visual/tool.dae" scale="0.019 0.019 0.019"/>>
+          <mesh filename="package://aescape_gazebo/meshes/visual/tool.dae" scale="0.019 0.019 0.019"/>
         </geometry>
       </visual>
       <collision>
         <geometry>
-          <mesh filename="package://aescape_gazebo/meshes/collision/tool.stl" scale="0.019 0.019 0.019"/>
+          <mesh filename="package://aescape_gazebo/meshes/visual/tool.stl" scale="0.019 0.019 0.019"/>
         </geometry>
       </collision>
       <inertial>
         <origin xyz="0 0 0" rpy="0 0 0"/>
-        <mass value="0.0"/>
-        <inertia ixx="0.001" ixy="0.0" ixz="0.0" iyy="0.001" iyz="0.0" izz="0.001"/>
+        <mass value="0.68"/>
+        <inertia ixx="0.1" ixy="0.0" ixz="0.0" iyy="0.1" iyz="0.0" izz="0.1"/>
       </inertial>
     </link>
-    <xacro:unless value="${connected_to == ''}">
-      <joint name="${robot_ns}_arm_tool_joint" type="fixed">
-        <parent link="${connected_to}"/>
-        <child link="${robot_ns}_arm_tool_link"/>
-        <origin xyz="${xyz}" rpy="${rpy}"/>
-        <axis xyz="0 0 1"/>
-      </joint>
-    </xacro:unless>
+    <joint name="${arm_id}_arm_joint_tool" type="fixed">
+      <parent link="${connected_to}"/>
+      <child link="${arm_id}_arm_tool_link"/>
+      <origin rpy="${rpy}" xyz="${xyz}"/>
+    </joint>
     <gazebo reference="${arm_id}_arm_tool_link">
       <material>Gazebo/Grey</material>

Commit message: fix: camera_bases positions updated

File: urdf/robot.urdf.xacro (robot description, xacro)
@@ -26,15 +26,4 @@
     <xacro:panda_transmission robot_name="left_arm" robot_ns="left"/>
     <xacro:panda_transmission robot_name="right_arm" robot_ns="right"/>
-    <!--
-    - parent: left_arm_base_link
-      child: left_camera_base
-      x: 0.1404396785274887
-      y: -0.05307111179809734
-      z: 1.358923271686402
-      qx: 0.8141408253648392
-      qy: -0.1035370936067316
-      qz: -0.5689034786331804
-      qw: 0.05294918214014413
-    -->
     <xacro:depth_camera
     camera_name="left_camera_base"
@@ -42,48 +31,14 @@
     xyz="0.1404396785274887 -0.05307111179809734 1.358923271686402"
     rpy="2.610 1.156 -0.605"/>
-    <!--
-    - Translation: [0.143, -0.021, 1.356]
-    - Rotation: in Quaternion [-0.716, -0.665, -0.052, -0.208]
-            in RPY (radian) [2.759, 0.204, 1.457]
-            in RPY (degree) [158.054, 11.677, 83.483]
-    -->
-    <link name="left_rgb_camera_link"/>
-    <joint name="left_arm_base_to_left_rgb_camera_joint" type="fixed">
-      <parent link="left_arm_base_link"/>
-      <child link="left_rgb_camera_link"/>
-      <origin xyz="0.143 -0.021 1.356" rpy="2.759 0.204 1.457" />
-    </joint>
-    <!--
-    - parent: left_rgb_camera_link
-      child: center_camera_base
-      x: 0.9361730730167426
-      y: 0.290787205870503
-      z: -0.01642135865139904
-      qx: -0.3264977374886928
-      qy: 0.7636580414712461
-      qz: -0.4407959649381484
-      qw: -0.340476950638661
-    -->
     <xacro:depth_camera
     camera_name="center_camera_base"
-    connected_to="left_rgb_camera_link"
-    xyz="0.9361730730167426 0.290787205870503 -0.01642135865139904"
-    rpy="-2.270 -0.941 -2.798"/>
-    <!--
-  - parent: left_rgb_camera_link
-    child: right_camera_base
-    x: 0.07076650529446413
-    y: 0.6961604567394116
-    z: 0.2631112375688656
-    qx: -0.3316925446975479
-    qy: -0.1864996386672192
-    qz: -0.6685085657833876
-    qw: 0.6389790561964096
-    -->
+    connected_to="left_arm_base_link"
+    xyz="0.512 0.885 1.288"
+    rpy="1.482 0.767 -1.520"/>
     <xacro:depth_camera
     camera_name="right_camera_base"
-    connected_to="left_rgb_camera_link"
-    xyz="0.07076650529446413 0.6961604567394116 0.2631112375688656"
-    rpy="-0.241 -0.750 -1.521"/>
+    connected_to="left_arm_base_link"
+    xyz="0.890 -0.033 1.358"
+    rpy="-2.960 1.106 -2.920"/>
   </xacro:if>
   <link name="table_center">

Commit message: feat: world link added to the robot model

File: urdf/robot.urdf.xacro (robot description, xacro)
@@ -89,5 +89,5 @@
     <parent link="table_center"/>
     <child link="table"/>
-  </joint> -->
+  </joint>
   <link name="canonical_body_origin"/>
   <joint name="canonical_body_joint" type="fixed">
@@ -101,4 +101,10 @@
     <parent link="table_center"/>
     <child link="canonical_smpl_origin"/>
+  </joint>-->
+  <link name="world"/>
+  <joint name="world_to_left_arm_base_link" type="fixed">
+    <parent link="world"/>
+    <child link="left_arm_base_link"/>
+    <origin xyz="0.0 0.0 0.0" rpy="0 0 0" />
   </joint>
 </robot>

Commit message: feat: pepe model added to robot

File: urdf/robot.urdf.xacro (robot description, xacro)
@@ -59,5 +59,5 @@
     </collision>
     <inertial>
-        <mass value="0.2"/>
+        <mass value="200"/>
         <inertia ixx="1.0" ixy="0.0" ixz="0.0" iyy="1.0" iyz="0.0" izz="1.0"/>
     </inertial>
@@ -108,3 +108,20 @@
     <origin xyz="0.0 0.0 0.0" rpy="0 0 0" />
   </joint>
+  <link name="pepe">
+    <visual>
+        <geometry>
+          <mesh filename="package://aescape_gazebo/models/pepe/meshes/pepe.dae"/>
+        </geometry>
+      </visual>
+      <collision>
+        <geometry>
+          <mesh filename="package://aescape_gazebo/models/pepe/meshes/pepe.dae"/>
+        </geometry>
+      </collision>
+  </link>
+  <joint name="pepe_to_world" type="fixed">
+   <parent link="world"/>
+    <child link="pepe"/>
+    <origin xyz="0.5 -1.2 0.40" rpy="${pi/2} 0 ${pi}" /> <!-- Default Values -->
+  </joint>
 </robot>

Commit message: feat: pepe link added

File: urdf/robot.urdf.xacro (robot description, xacro)
@@ -9,4 +9,10 @@
     <xacro:panda_arm arm_id="${arm_id}_arm" connected_to="${arm_id}_arm_base_link" in_gazebo="${use_gazebo}"  xyz="0 0 0" rpy="0 0 0"/>
   </xacro:macro>
+  <link name="world"/>
+  <joint name="world_to_left_arm_base_link" type="fixed">
+    <parent link="world"/>
+    <child link="left_arm_base_link"/>
+    <origin xyz="0.0 0.0 0.0" rpy="0 0 0" />
+  </joint>
   <joint name="right_arm_base_link_calibration" type="fixed">
     <parent link="left_arm_base_link"/>
@@ -22,4 +28,6 @@
     <xacro:include filename="$(find aescape_gazebo)/urdf/panda.transmission.xacro"/>
     <xacro:include filename="$(find aescape_gazebo)/urdf/depth_camera.xacro"/>
+    <xacro:include filename="$(find aescape_gazebo)/urdf/pepe.xacro"/>
+    <!--xacro:pepe name="pepe" connected_to="world" xyz="0.5 -1.4 0.45" rpy="${pi/2} 0.0 ${pi}"/-->
     <xacro:panda_gazebo arm_id="left"/>
     <xacro:panda_gazebo arm_id="right"/>
@@ -47,7 +55,4 @@
       	<box size="0.76 1.83 0.1"/>
       </geometry>
-      <!--material name="Grey">
-	      <color rgba="0.5 0.5 0.5 0.8"/>
-      </material-->
       <origin rpy="0 0 0" xyz="0 -0.6332 -0.05"/>
     </visual>
@@ -59,13 +64,13 @@
     </collision>
     <inertial>
-        <mass value="200"/>
-        <inertia ixx="1.0" ixy="0.0" ixz="0.0" iyy="1.0" iyz="0.0" izz="1.0"/>
+      <mass value="200"/>
+      <inertia ixx="1.0" ixy="0.0" ixz="0.0" iyy="1.0" iyz="0.0" izz="1.0"/>
     </inertial>
-    <gazebo reference="table_center">
-      <material>Gazebo/Black</material>
-      <mu1>0.2</mu1>
-      <mu2>0.2</mu2>
-    </gazebo>
   </link>
+  <gazebo reference="table_center">
+    <material>Gazebo/White</material>
+    <mu1>0.2</mu1>
+    <mu2>0.2</mu2>
+  </gazebo>
   <joint name="table_center_calibration" type="fixed">
     <parent link="left_arm_base_link"/>
@@ -102,26 +107,3 @@
     <child link="canonical_smpl_origin"/>
   </joint>-->
-  <link name="world"/>
-  <joint name="world_to_left_arm_base_link" type="fixed">
-    <parent link="world"/>
-    <child link="left_arm_base_link"/>
-    <origin xyz="0.0 0.0 0.0" rpy="0 0 0" />
-  </joint>
-  <link name="pepe">
-    <visual>
-        <geometry>
-          <mesh filename="package://aescape_gazebo/models/pepe/meshes/pepe.dae"/>
-        </geometry>
-      </visual>
-      <collision>
-        <geometry>
-          <mesh filename="package://aescape_gazebo/models/pepe/meshes/pepe.dae"/>
-        </geometry>
-      </collision>
-  </link>
-  <joint name="pepe_to_world" type="fixed">
-   <parent link="world"/>
-    <child link="pepe"/>
-    <origin xyz="0.5 -1.2 0.40" rpy="${pi/2} 0 ${pi}" /> <!-- Default Values -->
-  </joint>
 </robot>
