Commit message: feat: box models added

File: urdf/pepe.xacro (robot description, xacro)
@@ -14,4 +14,5 @@
       </collision>
       <inertial>
+        <origin xyz="0 0 0" rpy="0 0 0"/>
         <mass value="90"/>
         <inertia ixx="0.0" ixy="0.0" ixz="0.0" iyy="0.0" iyz="0.0" izz="0.0"/>
@@ -24,13 +25,13 @@
     </joint>
     <gazebo reference="${name}_link">
-      <!--material>Gazebo/Grey</material-->
-      <mu1 value="20000.0"/>
-      <mu2 value="20000.0"/>
-      <kp value="10000000.0" />
-      <kd value="1.0" />
-      <!--sensor name="${name}_contact" type="contact">
+      <mu1 value="0.2"/>
+      <mu2 value="0.2"/>
+      <kp value="10000000.0"/>
+      <kd value="1.0"/>
+      <selfCollide>true</selfCollide>
+      <sensor name="${name}_contact" type="contact">
         <always_on>true</always_on>
         <contact>
-          <collision>${name}_collision_1</collision>
+          <collision>${name}_link_collision</collision>
         </contact>
         <plugin name="${name}_plugin" filename="libgazebo_ros_bumper.so">
@@ -38,5 +39,5 @@
           <frameName>${name}_link</frameName>
         </plugin>
-      </sensor-->
+      </sensor>
     </gazebo>
   </xacro:macro>

File: urdf/robot.urdf (robot description, URDF)
Before this commit: robot aescape_robot, 28 links, 27 joints
Links:
- removed link canonical_body_origin
- removed link canonical_smpl_origin
- added link pepe_link, mass 90; collision mesh filename=package://aescape_gazebo/models/pepe/meshes/pepe.stl; visual mesh filename=package://aescape_gazebo/models/pepe/meshes/pepe.dae
- added link world
- link table_center: mass 0.2 -> 200
Joints:
- removed joint canonical_body_joint
- removed joint canonical_smpl_origin_joint
- added joint pepe_to_joint: type fixed, parent world, child pepe_link, origin xyz=0.5 -1.4 0.45 rpy=1.57079632679 0.0 3.14159265359
- added joint world_to_left_arm_base_link: type fixed, parent world, child left_arm_base_link, origin xyz=0.0 0.0 0.0 rpy=0 0 0

File: urdf/robot.urdf.xacro (robot description, xacro)
@@ -29,5 +29,5 @@
     <xacro:include filename="$(find aescape_gazebo)/urdf/depth_camera.xacro"/>
     <xacro:include filename="$(find aescape_gazebo)/urdf/pepe.xacro"/>
-    <!--xacro:pepe name="pepe" connected_to="world" xyz="0.5 -1.4 0.45" rpy="${pi/2} 0.0 ${pi}"/-->
+    <xacro:pepe name="pepe" connected_to="world" xyz="0.50 -1.20 0.30" rpy="${pi/2} 0.0 ${pi}"/>
     <xacro:panda_gazebo arm_id="left"/>
     <xacro:panda_gazebo arm_id="right"/>
@@ -64,5 +64,5 @@
     </collision>
     <inertial>
-      <mass value="200"/>
+      <mass value="2"/>
       <inertia ixx="1.0" ixy="0.0" ixz="0.0" iyy="1.0" iyz="0.0" izz="1.0"/>
     </inertial>
@@ -72,4 +72,5 @@
     <mu1>0.2</mu1>
     <mu2>0.2</mu2>
+    <selfCollide>true</selfCollide>
   </gazebo>
   <joint name="table_center_calibration" type="fixed">

File: urdf/tool.xacro (robot description, xacro)
@@ -28,4 +28,5 @@
       <mu1>0.2</mu1>
       <mu2>0.2</mu2>
+      <selfCollide>true</selfCollide>
       <sensor name="${arm_id}_arm_tool_contact" type="contact">
         <always_on>true</always_on>
